Commit message: feat: Adjust ur5 position in the world frame.

File: src/Universal_Robots_ROS2_Description/urdf/ur.urdf.xacro (robot description, xacro)
@@ -115,5 +115,5 @@
      trajectory_port="$(arg trajectory_port)"
      >
-     <origin xyz="0 0 0" rpy="0 0 0" />          <!-- position robot in the world -->
+     <origin xyz="0 0 0" rpy="0 0 -3.92699" />          <!-- position robot in the world -->
    </xacro:ur_robot>
    <xacro:if value="$(arg sim_gazebo)">

Commit message: feat: Add racket frame in the ur description.

File: src/Universal_Robots_ROS2_Description/urdf/ur.urdf.xacro (robot description, xacro)
@@ -117,5 +117,47 @@
      <origin xyz="0 0 0" rpy="0 0 -3.92699" />          <!-- position robot in the world -->
    </xacro:ur_robot>
-   <xacro:if value="$(arg sim_gazebo)">
+  <link name="racket">
+    <visual>
+      <geometry>
+        <cylinder radius="0.08" length="0.01"/>
+      </geometry>
+      <material name="racket_red">
+        <color rgba="0.8 0.1 0.1 1"/>
+      </material>
+      <origin xyz="0 0 0" rpy="0 0 0"/>
+    </visual>
+    <collision>
+      <geometry>
+        <cylinder radius="0.08" length="0.01"/>
+      </geometry>
+      <origin xyz="0 0 0" rpy="0 0 0"/>
+    </collision>
+    <visual>
+      <geometry>
+        <cylinder radius="0.015" length="0.10"/>
+      </geometry>
+      <material name="handle">
+        <color rgba="0 0 0 1"/>
+      </material>
+      <origin xyz="-0.13 0 0" rpy="0 1.5708 0"/>
+    </visual>
+    <collision>
+      <geometry>
+        <cylinder radius="0.015" length="0.10"/>
+      </geometry>
+      <origin xyz="-0.13 0 0" rpy="0 1.5708 0"/>
+    </collision>
+    <inertial>
+      <mass value="0.25"/>
+      <origin xyz="0 0 0"/>
+      <inertia ixx="0.0" ixy="0.0" ixz="0.0" iyy="0.0" iyz="0.0" izz="0.0"/>
+    </inertial>
+  </link>
+  <joint name="tool0_to_racket" type="fixed">
+    <parent link="$(arg tf_prefix)tool0"/>
+    <child link="racket"/>
+    <origin xyz="0 0 0.20" rpy="0 -1.57 0"/>
+  </joint>
+  <xacro:if value="$(arg sim_gazebo)">
     <!-- Gazebo plugins -->
     <gazebo reference="world">

Commit message: fix: Update racket dimension and position.

File: src/Universal_Robots_ROS2_Description/urdf/ur.urdf.xacro (robot description, xacro)
@@ -120,5 +120,5 @@
     <visual>
       <geometry>
-        <cylinder radius="0.08" length="0.01"/>
+        <cylinder radius="0.075" length="0.01"/>
       </geometry>
       <material name="racket_red">
@@ -129,5 +129,5 @@
     <collision>
       <geometry>
-        <cylinder radius="0.08" length="0.01"/>
+        <cylinder radius="0.075" length="0.01"/>
       </geometry>
       <origin xyz="0 0 0" rpy="0 0 0"/>
@@ -140,5 +140,5 @@
         <color rgba="0 0 0 1"/>
       </material>
-      <origin xyz="-0.13 0 0" rpy="0 1.5708 0"/>
+      <origin xyz="-0.12 0 0" rpy="0 1.5708 0"/>
     </visual>
     <collision>
@@ -146,5 +146,5 @@
         <cylinder radius="0.015" length="0.10"/>
       </geometry>
-      <origin xyz="-0.13 0 0" rpy="0 1.5708 0"/>
+      <origin xyz="-0.12 0 0" rpy="0 1.5708 0"/>
     </collision>
     <inertial>
@@ -157,5 +157,5 @@
     <parent link="$(arg tf_prefix)tool0"/>
     <child link="racket"/>
-    <origin xyz="0 0 0.20" rpy="0 -1.57 0"/>
+    <origin xyz="0 0 0.19" rpy="1.57 -1.57 0"/>
   </joint>
   <xacro:if value="$(arg sim_gazebo)">

Commit message: feat: Add calibration_plate frame in UR5 urdf.

File: src/Universal_Robots_ROS2_Description/urdf/ur.urdf.xacro (robot description, xacro)
@@ -159,4 +159,30 @@
     <origin xyz="0 0 0.19" rpy="1.57 -1.57 0"/>
   </joint>
+  <link name="calibration_plate">
+    <!-- <visual>
+      <geometry>
+        <box size="0.1 0.1 0.005"/>
+      </geometry>
+      <material name="plate_grey">
+        <color rgba="0.5 0.5 0.5 1"/>
+      </material>
+      <origin xyz="0 0 0" rpy="0 0 0"/>
+    </visual>
+    <collision>
+      <geometry>
+        <box size="0.1 0.1 0.005"/>
+      </geometry>
+      <origin xyz="0 0 0" rpy="0 0 0"/>
+    </collision>
+    <inertial>
+      <mass value="0.0"/> <origin xyz="0 0 0"/>
+      <inertia ixx="0.0" ixy="0.0" ixz="0.0" iyy="0.0" iyz="0.0" izz="0.0"/>
+    </inertial> -->
+  </link>
+  <joint name="tool0_to_calibration_plate" type="fixed">
+    <parent link="$(arg tf_prefix)tool0"/>
+    <child link="calibration_plate"/>
+    <origin xyz="0 0 0.06" rpy="0 0 0"/>
+  </joint>
   <xacro:if value="$(arg sim_gazebo)">
     <!-- Gazebo plugins -->

Commit message: feat: Remove the racket urdf and include the rg2 gripper.

File: src/Universal_Robots_ROS2_Description/urdf/ur.urdf.xacro (robot description, xacro)
@@ -117,48 +117,11 @@
      <origin xyz="0 0 0" rpy="0 0 -3.92699" />          <!-- position robot in the world -->
    </xacro:ur_robot>
-  <link name="racket">
+  <xacro:include filename="$(find onrobot_rg2_description)/urdf/onrobot_rg2.urdf.xacro" ns="gripper" />
+  <xacro:gripper.onrobot_rg2
+    parent_link="tool0"
+    xyz="0.0 0.0 0.0"
+    rpy="0.0 ${-pi/2} ${pi/2}" />
+  <!-- <link name="calibration_plate">
     <visual>
-      <geometry>
-        <cylinder radius="0.075" length="0.01"/>
-      </geometry>
-      <material name="racket_red">
-        <color rgba="0.8 0.1 0.1 1"/>
-      </material>
-      <origin xyz="0 0 0" rpy="0 0 0"/>
-    </visual>
-    <collision>
-      <geometry>
-        <cylinder radius="0.075" length="0.01"/>
-      </geometry>
-      <origin xyz="0 0 0" rpy="0 0 0"/>
-    </collision>
-    <visual>
-      <geometry>
-        <cylinder radius="0.015" length="0.10"/>
-      </geometry>
-      <material name="handle">
-        <color rgba="0 0 0 1"/>
-      </material>
-      <origin xyz="-0.12 0 0" rpy="0 1.5708 0"/>
-    </visual>
-    <collision>
-      <geometry>
-        <cylinder radius="0.015" length="0.10"/>
-      </geometry>
-      <origin xyz="-0.12 0 0" rpy="0 1.5708 0"/>
-    </collision>
-    <inertial>
-      <mass value="0.25"/>
-      <origin xyz="0 0 0"/>
-      <inertia ixx="0.0" ixy="0.0" ixz="0.0" iyy="0.0" iyz="0.0" izz="0.0"/>
-    </inertial>
-  </link>
-  <joint name="tool0_to_racket" type="fixed">
-    <parent link="$(arg tf_prefix)tool0"/>
-    <child link="racket"/>
-    <origin xyz="0 0 0.19" rpy="1.57 -1.57 0"/>
-  </joint>
-  <link name="calibration_plate">
-    <!-- <visual>
       <geometry>
         <box size="0.1 0.1 0.005"/>
@@ -178,5 +141,5 @@
       <mass value="0.0"/> <origin xyz="0 0 0"/>
       <inertia ixx="0.0" ixy="0.0" ixz="0.0" iyy="0.0" iyz="0.0" izz="0.0"/>
-    </inertial> -->
+    </inertial>
   </link>
   <joint name="tool0_to_calibration_plate" type="fixed">
@@ -184,5 +147,5 @@
     <child link="calibration_plate"/>
     <origin xyz="0 0 0.06" rpy="0 0 0"/>
-  </joint>
+  </joint> -->
   <xacro:if value="$(arg sim_gazebo)">
     <!-- Gazebo plugins -->
